File: sensores.sch (KiCad schematic (older format))
At the start: 10 parts, among them J10 Conn_01x07_Female, J11 Conn_01x03_Female, J12 Conn_02x20_Odd_Even, J4 Conn_01x06_Male, J5 Conn_01x06_Male, J6 Conn_01x06_Male, J7 Conn_01x06_Male, J8 Conn_01x06_Male, J9 Conn_01x06_Male, U4 DHT11

Commit message: Adicionando radio LoRa. Criando um .sch para a Raspberry e para o radio
Parts:
- removed J10: Conn_01x07_Female, Connector_Harwin:Harwin_M20-89007xx_1x07_P2.54mm_Horizontal, symbol Connector:Conn_01x07_Female
- removed J12: Conn_02x20_Odd_Even, Connector_PinHeader_2.54mm:PinHeader_2x20_P2.54mm_Vertical, symbol Connector_Generic:Conn_02x20_Odd_Even
Connections:
- net labels added: DHT_OUTPUT
- net labels removed: DHT_OUT, RASP_INT0, RASP_INT1, RASP_S0, RASP_S1, RASP_S2, RASP_S3, RASP_SCL0, RASP_SCL1, RASP_SDA0, RASP_SDA1, SPI0_CLK, SPI0_MISO, SPI0_MOSI, UART_RX, UART_TX
- wire segments 72 -> 67
- no-connect marks 7 -> 0
Other:
- note removed: "SDS011"
