File: rfm952.sch (KiCad schematic (older format))
At the start: 3 parts, among them J13 5-1814400-1, U7 RFM95W-915S2

Commit message: Versão v0 finalizada. Adiciona pasta para os arquivos de saída e de fabricacao.
Parts:
- U7: footprint RF_Module:HOPERF_RFM9XW_SMD -> RF_Module:HOPERF_RFM9XW_THT
Changed lines of the file:
@@
 $Descr A4 11693 8268
 encoding utf-8
-Sheet 7 7
+Sheet 6 7
 Title ""
 Date ""
@@
 F 0 "U7" H 5250 4681 50  0000 C CNN
 F 1 "RFM95W-915S2" H 5250 4590 50  0000 C CNN
-F 2 "RF_Module:HOPERF_RFM9XW_SMD" H 1950 5650 50  0001 C CNN
+F 2 "RF_Module:HOPERF_RFM9XW_THT" H 1950 5650 50  0001 C CNN
 F 3 "https://www.hoperf.com/data/upload/portal/20181127/5bfcbea20e9ef.pdf" H 1950 5650 50  0001 C CNN
 	1    5250 4000
