File: regulators.sch (KiCad schematic (older format))
At the start: 9 parts, among them U1 LM7805_TO220, U2 LM1117-3.3

Commit message: Conexão entre os componentes. Correção da lib do buck-boost. Separação do 3v3 da raspberry e do 3v3 do regulador
Parts:
- removed U?: BUCK_BOOST_BOARD, 22-23-2061:DIP-4_1889_ELL, symbol Battery_Management_bq:BUCK_BOOST_BOARD
- added U8: BUCK_BOOST_BOARD, symbol Battery_Management_2:BUCK_BOOST_BOARD
Changed lines of the file:
@@
 $EndDescr
-$Comp
-L Battery_Management_bq:BUCK_BOOST_BOARD U?
-U 1 1 61C62395
-P 2050 2500
-F 0 "U?" H 2050 2525 50  0000 C CNN
-F 1 "BUCK_BOOST_BOARD" H 2050 2434 50  0000 C CNN
-F 2 "22-23-2061:DIP-4_1889_ELL" H 2050 2500 50  0001 C CNN
-F 3 "" H 2050 2500 50  0001 C CNN
-	1    2050 2500
-	1    0    0    -1
-$EndComp
 $Comp
 L power:GND #PWR0106
@@
 9V_BUCK_BOOST
 Wire Wire Line
+	4900 2650 5050 2650
+$Comp
+L Battery_Management_2:BUCK_BOOST_BOARD U8
+U 1 1 61FDE5BF
+P 2050 2500
+F 0 "U8" H 2050 2525 50  0000 C CNN
+F 1 "BUCK_BOOST_BOARD" H 2050 2434 50  0000 C CNN
+F 2 "" H 2050 2500 50  0001 C CNN
+F 3 "" H 2050 2500 50  0001 C CNN
+	1    2050 2500
+	1    0    0    -1
+$EndComp
+Wire Wire Line
 	8400 2700 8600 2700
-Wire Wire Line
-	4900 2650 5050 2650
 $EndSCHEMATC

Commit message: Roteamento da PCB pronto; Agora o 3v3 da raspberry alimenta os resistores de pull up da comunicacao i2c do bq24160
Parts:
- U8: footprint (none) -> 22-23-2061:DIP-4_1889_ELL
Changed lines of the file:
@@
 F 0 "U8" H 2050 2525 50  0000 C CNN
 F 1 "BUCK_BOOST_BOARD" H 2050 2434 50  0000 C CNN
-F 2 "" H 2050 2500 50  0001 C CNN
+F 2 "22-23-2061:DIP-4_1889_ELL" H 2050 2500 50  0001 C CNN
 F 3 "" H 2050 2500 50  0001 C CNN
 	1    2050 2500

Commit message: v3
Parts:
- renumbered U8 to U1, U1 to U2, U2 to U3
Changed lines of the file:
@@
 $Descr A4 11693 8268
 encoding utf-8
-Sheet 3 7
+Sheet 2 7
 Title ""
 Date "2021-12-26"
@@
 $EndDescr
 $Comp
-L power:GND #PWR0106
+L power:GND #PWR02
 U 1 1 61C78244
 P 1650 2950
-F 0 "#PWR0106" H 1650 2700 50  0001 C CNN
+F 0 "#PWR02" H 1650 2700 50  0001 C CNN
 F 1 "GND" H 1655 2777 50  0000 C CNN
 F 2 "" H 1650 2950 50  0001 C CNN
@@
 	1650 2900 1650 2950
 $Comp
-L power:GND #PWR0107
+L power:GND #PWR03
 U 1 1 61C78732
 P 2450 2950
-F 0 "#PWR0107" H 2450 2700 50  0001 C CNN
+F 0 "#PWR03" H 2450 2700 50  0001 C CNN
 F 1 "GND" H 2455 2777 50  0000 C CNN
 F 2 "" H 2450 2950 50  0001 C CNN
@@
 	2350 2750 2450 2750
 $Comp
-L Regulator_Linear:LM7805_TO220 U1
+L Regulator_Linear:LM7805_TO220 U2
 U 1 1 61C7A55C
 P 5700 2650
-F 0 "U1" H 5700 2892 50  0000 C CNN
+F 0 "U2" H 5700 2892 50  0000 C CNN
 F 1 "LM7805_TO220" H 5700 2801 50  0000 C CNN
 F 2 "Package_TO_SOT_THT:TO-220-3_Vertical" H 5700 2875 50  0001 C CIN
@@
 $EndComp
 $Comp
-L Regulator_Linear:LM1117-3.3 U2
+L Regulator_Linear:LM1117-3.3 U3
 U 1 1 61C7CD12
 P 9250 2700
-F 0 "U2" H 9250 2942 50  0000 C CNN
+F 0 "U3" H 9250 2942 50  0000 C CNN
 F 1 "LM1117-3.3" H 9250 2851 50  0000 C CNN
 F 2 "Package_TO_SOT_THT:TO-220-3_Vertical" H 9250 2700 50  0001 C CNN
@@
 $EndComp
 $Comp
-L power:GND #PWR0108
+L power:GND #PWR04
 U 1 1 61C81AFD
 P 5050 3150
-F 0 "#PWR0108" H 5050 2900 50  0001 C CNN
+F 0 "#PWR04" H 5050 2900 50  0001 C CNN
 F 1 "GND" H 5055 2977 50  0000 C CNN
 F 2 "" H 5050 3150 50  0001 C CNN
@@
 $EndComp
 $Comp
-L power:GND #PWR0109
+L power:GND #PWR05
 U 1 1 61C82072
 P 6300 3150
-F 0 "#PWR0109" H 6300 2900 50  0001 C CNN
+F 0 "#PWR05" H 6300 2900 50  0001 C CNN
 F 1 "GND" H 6305 2977 50  0000 C CNN
 F 2 "" H 6300 3150 50  0001 C CNN
@@
 $EndComp
 $Comp
-L power:GND #PWR0110
+L power:GND #PWR07
 U 1 1 61C90E26
 P 8600 3200
-F 0 "#PWR0110" H 8600 2950 50  0001 C CNN
+F 0 "#PWR07" H 8600 2950 50  0001 C CNN
 F 1 "GND" H 8605 3027 50  0000 C CNN
 F 2 "" H 8600 3200 50  0001 C CNN
@@
 $EndComp
 $Comp
-L power:GND #PWR0111
+L power:GND #PWR08
 U 1 1 61C90E2C
 P 9850 3200
-F 0 "#PWR0111" H 9850 2950 50  0001 C CNN
+F 0 "#PWR08" H 9850 2950 50  0001 C CNN
 F 1 "GND" H 9855 3027 50  0000 C CNN
 F 2 "" H 9850 3200 50  0001 C CNN
@@
 Connection ~ 9850 2700
 $Comp
-L power:+5V #PWR0112
+L power:+5V #PWR06
 U 1 1 61C8CB6E
 P 6500 2600
-F 0 "#PWR0112" H 6500 2450 50  0001 C CNN
+F 0 "#PWR06" H 6500 2450 50  0001 C CNN
 F 1 "+5V" H 6515 2773 50  0000 C CNN
 F 2 "" H 6500 2600 50  0001 C CNN
@@
 	6300 2650 6500 2650
 $Comp
-L power:+3.3V #PWR0113
+L power:+3.3V #PWR09
 U 1 1 61C8DFF5
 P 10050 2600
-F 0 "#PWR0113" H 10050 2450 50  0001 C CNN
+F 0 "#PWR09" H 10050 2450 50  0001 C CNN
 F 1 "+3.3V" H 10065 2773 50  0000 C CNN
 F 2 "" H 10050 2600 50  0001 C CNN
@@
 	4900 2650 5050 2650
 $Comp
-L Battery_Management_2:BUCK_BOOST_BOARD U8
+L Battery_Management_2:BUCK_BOOST_BOARD U1
 U 1 1 61FDE5BF
 P 2050 2500
-F 0 "U8" H 2050 2525 50  0000 C CNN
+F 0 "U1" H 2050 2525 50  0000 C CNN
 F 1 "BUCK_BOOST_BOARD" H 2050 2434 50  0000 C CNN
 F 2 "22-23-2061:DIP-4_1889_ELL" H 2050 2500 50  0001 C CNN
