File: envcity_aqm_v2.kicad_sch (KiCad schematic)
At the start: 137 parts, among them IC1 DS1307ZN+, IC2 DMMT5401-7F, IC3 DMMT5401-7F, IC4 DMMT5401-7-F, IC5 ESP32-S2-SOLO-N4R2, J1 Conn_01x06_Male, J10 Conn_01x03_Male, J11 Conn_01x04_Male, J12 Conn_01x02_Male, J13 Conn_01x02_Male, J14 Micro_SD_Card, J15 Conn_01x08_Pin, J2 Screw_Terminal_01x02, J3 Screw_Terminal_01x02, J4 Conn_01x06_Male, J5 Conn_01x06_Male, J6 Conn_01x06_Male, J7 Conn_01x06_Male, J8 USB_B_Micro, J9 Conn_01x06_Male, Q1 DMG2301L, Q12 DMG2301L / DMP2045U, Q13 DMN10H220L, Q14 DMN10H220L, Q2 DMG2301L, Q5 DMG2301L / DMP2045U, Q8 DMG2301L, Q9 DMG2301L / DMP2045U, SW1 BOOT, SW1 RESET, U1 ADS1115IDGS, U10 RFM95W-915S2, U11 AP2112K-3.3, U2 CD74HC4067M, U3 AP2112K-3.3, U4 LM2596S-5, U5 TP4056, U6 MT3608, U7 MT3608, U8 DHT11, U9 USBLC6-2SC6, Y1 32,768KHz

Commit message: Add um monte de coisa
Parts:
- removed D3: 5V, Diode_SMD:D_SOD-323, symbol envcity_aqm_v2-rescue:D_Zener_ALT-Device
- removed IC5: ESP32-S2-SOLO-N4R2, ESP32S2SOLON4R2, symbol ESP32-S2-SOLO-N4R2:ESP32-S2-SOLO-N4R2
- removed R15: 1K, Resistor_SMD:R_0805_2012Metric_Pad1.15x1.40mm_HandSolder, symbol Device:R
- added C17: 100nF, Capacitor_SMD:C_0805_2012Metric, symbol Device:C_Small
- added IC6: ESP32-S2-SOLO-N4R2, ESP32-S2-SOLO-N4R2:ESP32S2SOLON4R2, symbol ESP32-S2-SOLO-N4R2:ESP32-S2-SOLO-N4R2
- added J7: Conn_01x06_Pin, Connector_Molex:Molex_KK-254_AE-6410-06A_1x06_P2.54mm_Vertical, symbol Connector:Conn_01x06_Pin
- AE1: footprint (none) -> Connector_Coaxial:U.FL_Molex_MCRF_73412-0110_Vertical
- C1: renamed from C22; footprint Capacitor_SMD:C_0805_2012Metric_Pad1.15x1.40mm_HandSolder -> Capacitor_SMD:C_0805_2012Metric
- C11: renamed from C5; footprint Capacitor_SMD:C_0603_1608Metric -> Capacitor_SMD:C_0805_2012Metric
- C12: renamed from C20; footprint Capacitor_SMD:C_0805_2012Metric_Pad1.15x1.40mm_HandSolder -> Capacitor_SMD:C_0805_2012Metric
- C13: renamed from C14; footprint Capacitor_SMD:C_0805_2012Metric_Pad1.15x1.40mm_HandSolder -> Capacitor_SMD:C_0805_2012Metric
- C18: renamed from C16; footprint Capacitor_SMD:C_0805_2012Metric_Pad1.15x1.40mm_HandSolder -> Capacitor_SMD:C_0805_2012Metric
- C19: renamed from C28; footprint Capacitor_SMD:C_0805_2012Metric_Pad1.15x1.40mm_HandSolder -> Capacitor_SMD:C_0805_2012Metric
- C2: renamed from C23; footprint Capacitor_SMD:C_0805_2012Metric_Pad1.15x1.40mm_HandSolder -> Capacitor_SMD:C_0805_2012Metric
- C20: renamed from C12; footprint Capacitor_SMD:C_0805_2012Metric_Pad1.15x1.40mm_HandSolder -> Capacitor_SMD:C_0805_2012Metric
- C21: renamed from C30; footprint Capacitor_SMD:C_0805_2012Metric_Pad1.15x1.40mm_HandSolder -> Capacitor_SMD:C_0805_2012Metric
- C22: renamed from C31; footprint Capacitor_SMD:C_0603_1608Metric -> Capacitor_SMD:C_0805_2012Metric
- C23: renamed from C32; footprint Capacitor_SMD:C_0603_1608Metric -> Capacitor_SMD:C_0805_2012Metric
- C24: renamed from C33; footprint Capacitor_SMD:C_0603_1608Metric -> Capacitor_SMD:C_0805_2012Metric
- C25: renamed from C17; footprint Capacitor_SMD:C_0805_2012Metric_Pad1.15x1.40mm_HandSolder -> Capacitor_SMD:C_0805_2012Metric
- C26: renamed from C29; footprint Capacitor_SMD:C_0805_2012Metric_Pad1.15x1.40mm_HandSolder -> Capacitor_SMD:C_0805_2012Metric
- C27: renamed from C13; footprint Capacitor_SMD:C_0805_2012Metric_Pad1.15x1.40mm_HandSolder -> Capacitor_SMD:C_0805_2012Metric
- C28: renamed from C1; footprint Capacitor_SMD:C_0805_2012Metric_Pad1.15x1.40mm_HandSolder -> Capacitor_SMD:C_0805_2012Metric
- C29: renamed from C25; footprint (none) -> Capacitor_SMD:C_0805_2012Metric
- C3: renamed from C9; footprint Capacitor_SMD:C_0805_2012Metric_Pad1.15x1.40mm_HandSolder -> Capacitor_SMD:C_0805_2012Metric
- C30: renamed from C24; footprint (none) -> Capacitor_SMD:C_0805_2012Metric
- C31: renamed from C19; footprint (none) -> Capacitor_SMD:C_0805_2012Metric
- C32: renamed from C3; footprint (none) -> Capacitor_SMD:C_0805_2012Metric
- C33: renamed from C18; footprint (none) -> Capacitor_SMD:C_0805_2012Metric
- C34: renamed from C2; footprint Capacitor_SMD:C_0805_2012Metric_Pad1.15x1.40mm_HandSolder -> Capacitor_SMD:C_0805_2012Metric
- C4: renamed from C10; footprint Capacitor_SMD:C_0805_2012Metric_Pad1.15x1.40mm_HandSolder -> Capacitor_SMD:C_0805_2012Metric
- C5: renamed from C11; footprint Capacitor_SMD:C_0805_2012Metric_Pad1.15x1.40mm_HandSolder -> Capacitor_SMD:C_0805_2012Metric
- C6: renamed from C4; footprint (none) -> Capacitor_SMD:C_0603_1608Metric
- C7: renamed from C6; footprint (none) -> Capacitor_SMD:C_0603_1608Metric
- C8: renamed from C21; footprint Capacitor_SMD:C_0805_2012Metric_Pad1.15x1.40mm_HandSolder -> Capacitor_SMD:C_0805_2012Metric
- C9: renamed from C15; footprint Capacitor_SMD:C_0805_2012Metric_Pad1.15x1.40mm_HandSolder -> Capacitor_SMD:C_0805_2012Metric
- J1: renamed from J8; footprint (none) -> Connector_USB:USB_Micro-B_Wuerth_629105150521
- J14: renamed from J15; footprint (none) -> Connector_PinSocket_2.54mm:PinSocket_1x08_P2.54mm_Vertical_SMD_Pin1Left
- R1: renamed from R24; footprint Resistor_SMD:R_0805_2012Metric_Pad1.15x1.40mm_HandSolder -> Resistor_SMD:R_0805_2012Metric
- R10: renamed from R30; footprint Resistor_SMD:R_0603_1608Metric -> Resistor_SMD:R_0805_2012Metric
- R11: renamed from R32; footprint Resistor_SMD:R_0805_2012Metric_Pad1.15x1.40mm_HandSolder -> Resistor_SMD:R_0805_2012Metric
- R12: renamed from R33; footprint Resistor_SMD:R_0805_2012Metric_Pad1.15x1.40mm_HandSolder -> Resistor_SMD:R_0805_2012Metric
- R13: renamed from R26; footprint Resistor_SMD:R_0805_2012Metric_Pad1.15x1.40mm_HandSolder -> Resistor_SMD:R_0805_2012Metric
- R14: renamed from R27; footprint Resistor_SMD:R_0805_2012Metric_Pad1.15x1.40mm_HandSolder -> Resistor_SMD:R_0805_2012Metric
- R15: renamed from R7; footprint Resistor_SMD:R_0805_2012Metric_Pad1.15x1.40mm_HandSolder -> Resistor_SMD:R_0805_2012Metric
- R16: renamed from R21; footprint Resistor_SMD:R_0805_2012Metric_Pad1.15x1.40mm_HandSolder -> Resistor_SMD:R_0805_2012Metric
- R17: renamed from R31; footprint Resistor_SMD:R_0805_2012Metric_Pad1.15x1.40mm_HandSolder -> Resistor_SMD:R_0805_2012Metric
- R18: renamed from R25; footprint Resistor_SMD:R_0805_2012Metric_Pad1.15x1.40mm_HandSolder -> Resistor_SMD:R_0805_2012Metric
- R19: renamed from R8; footprint Resistor_SMD:R_0805_2012Metric_Pad1.15x1.40mm_HandSolder -> Resistor_SMD:R_0805_2012Metric
- R2: renamed from R22; footprint Resistor_SMD:R_0805_2012Metric_Pad1.15x1.40mm_HandSolder -> Resistor_SMD:R_0805_2012Metric
- R20: renamed from R9; footprint Resistor_SMD:R_0805_2012Metric_Pad1.15x1.40mm_HandSolder -> Resistor_SMD:R_0805_2012Metric
- R21: renamed from R10; footprint Resistor_SMD:R_0805_2012Metric_Pad1.15x1.40mm_HandSolder -> Resistor_SMD:R_0805_2012Metric
- R22: renamed from R36; footprint Resistor_SMD:R_0603_1608Metric -> Resistor_SMD:R_0805_2012Metric
- R23: renamed from R37; footprint Resistor_SMD:R_0603_1608Metric -> Resistor_SMD:R_0805_2012Metric
- R24: renamed from R16; footprint Resistor_SMD:R_0805_2012Metric_Pad1.15x1.40mm_HandSolder -> Resistor_SMD:R_0805_2012Metric
- R25: renamed from R6; footprint Resistor_SMD:R_0805_2012Metric_Pad1.15x1.40mm_HandSolder -> Resistor_SMD:R_0805_2012Metric
- R26: renamed from R3; footprint Resistor_SMD:R_0805_2012Metric_Pad1.15x1.40mm_HandSolder -> Resistor_SMD:R_0805_2012Metric
- R27: renamed from R17; footprint Resistor_SMD:R_0805_2012Metric_Pad1.15x1.40mm_HandSolder -> Resistor_SMD:R_0805_2012Metric
- R28: renamed from R34; footprint (none) -> Resistor_SMD:R_0805_2012Metric
- R29: renamed from R35; footprint (none) -> Resistor_SMD:R_0805_2012Metric
- R3: renamed from R23; footprint Resistor_SMD:R_0805_2012Metric_Pad1.15x1.40mm_HandSolder -> Resistor_SMD:R_0805_2012Metric
- R30: renamed from R11; footprint Resistor_SMD:R_0805_2012Metric_Pad1.15x1.40mm_HandSolder -> Resistor_SMD:R_0805_2012Metric
- R31: renamed from R12; footprint Resistor_SMD:R_0805_2012Metric_Pad1.15x1.40mm_HandSolder -> Resistor_SMD:R_0805_2012Metric
- R32: renamed from R13; footprint Resistor_SMD:R_0805_2012Metric_Pad1.15x1.40mm_HandSolder -> Resistor_SMD:R_0805_2012Metric
- R33: renamed from R14; footprint Resistor_SMD:R_0805_2012Metric_Pad1.15x1.40mm_HandSolder -> Resistor_SMD:R_0805_2012Metric
- R34: renamed from R28; footprint (none) -> Resistor_SMD:R_0805_2012Metric
- R35: renamed from R19; footprint (none) -> Resistor_SMD:R_0805_2012Metric
- R36: renamed from R20; footprint (none) -> Resistor_SMD:R_0805_2012Metric
- R37: renamed from R2; footprint Resistor_SMD:R_0805_2012Metric_Pad1.15x1.40mm_HandSolder -> Resistor_SMD:R_0805_2012Metric
- R5: renamed from R18; footprint Resistor_SMD:R_0805_2012Metric_Pad1.15x1.40mm_HandSolder -> Resistor_SMD:R_0805_2012Metric
- R6: renamed from R4; footprint (none) -> Resistor_SMD:R_0603_1608Metric
- R7: renamed from R5; footprint (none) -> Resistor_SMD:R_0603_1608Metric
- R8: renamed from R29; footprint Resistor_SMD:R_0603_1608Metric -> Resistor_SMD:R_0805_2012Metric
- R9: renamed from R1; footprint Resistor_SMD:R_0805_2012Metric_Pad1.15x1.40mm_HandSolder -> Resistor_SMD:R_0805_2012Metric
- U10: footprint (none) -> Connector_JAE:JAE_LY20-16P-DLT1_2x08_P2.00mm_Horizontal
- renumbered C7 to C10, C8 to C14, C26 to C15, C27 to C16, D4 to D1, D13 to D10, D9 to D12, D10 to D13, D12 to D15, D6 to D2, D7 to D3, D8 to D4, D5 to D6, D15 to D7, D1 to D8, D2 to D9, H3 to H2, H2 to H3, J6 to J10, J7 to J11, J1 to J12, J9 to J13, J12 to J15, J13 to J16, J14 to J4, J10 to J5, J11 to J6, J4 to J8, J5 to J9, L3 to L1, L1 to L3, Q9 to Q1, Q12 to Q2, Q1 to Q3, Q2 to Q4, Q8 to Q6, Q13 to Q7, Q14 to Q8, U5 to U1, U1 to U11, U9 to U2, U7 to U3, U6 to U4, U4 to U5, U11 to U6, U8 to U7, U3 to U8, U2 to U9
Connections:
- net +3V3: now also IC6.2 (3V3), J7.2 (Pin_2)
- net +5V: now also C17.1, J7.1 (Pin_1)
- net AIN1: now also J7.3 (Pin_3)
- net AIN2: now also J7.4 (Pin_4)
- net AIN3: now also J7.5 (Pin_5)
- net DHT_PIN: now also IC6.35 (IO42)
- net EN: now also IC6.3 (EN)
- net ESP_USB_D+: now also IC6.14 (IO20)
- net ESP_USB_D-: now also IC6.13 (IO19)
- net FAN1: now also IC6.38 (IO2)
- net FAN2: now also IC6.39 (IO1)
- net GND: now also Q1.1 (G), C17.2, IC6.1 (GND_1), IC6.40 (GND_2), IC6.41 (GND_3), IC6.42 (GND_4), IC6.43 (GND_5), IC6.44 (GND_6), IC6.45 (GND_7), IC6.46 (GND_8), IC6.47 (GND_9), IC6.48 (GND_10), IC6.49 (GND_11), J7.6 (Pin_6)
- net PMS_RX: now also IC6.37 (TXD0)
- net PMS_TX: now also IC6.36 (RXD0)
- net RFM_CS: now also IC6.21 (IO13)
- net RFM_DIO0: now also IC6.23 (IO21)
- net RFM_DIO1: now also IC6.24 (IO33)
- net RFM_DIO2: now also IC6.25 (IO34)
- net RFM_MISO: now also IC6.18 (IO10)
- net RFM_MOSI: now also IC6.19 (IO11)
- net RFM_RST: now also IC6.22 (IO14)
- net RFM_SCK: now also IC6.20 (IO12)
- net S0: now also IC6.4 (IO4)
- net S1: now also IC6.5 (IO5)
- net S2: now also IC6.6 (IO6)
- net S3: now also IC6.7 (IO7)
- net SCL: now also IC6.32 (IO39)
- net SDA: now also IC6.31 (IO38)
- net SD_CS: now also IC6.10 (IO17)
- net SD_MISO: now also IC6.9 (IO16)
- net SD_MOSI: now also IC6.8 (IO15)
- net SD_SCK: now also IC6.11 (IO18)
- net out_LM2596S: now reaches D12.1, L3.2, U5.2 (OUT)
- net at SW1.1: now also IC6.27 (IO0)
- no-connect marks 15 -> 23
Other:
- note added: "* Verificar simulações Power-Path * Alterar transitors para o DMMT - OK * Alterações Marcio: * Entradas analógicas an1...an3 expostas * Adicionado + 2 conectores p/ alphasense * Falta expor ANx... * ESP32-C3 - ok * Dissipador onboard - OK * Regulador 3V3 - OK * Um regulador para o esp32 e um para o rfm * ADD PMS5003 - ok"
- note added: "GP Analog inputs and Power Source"
- note removed: "* Verificar simulações Power-Path * Alterar transitors para o DMMT - OK * Alterações Marcio: * Entradas analógicas an1...an3 expostas * Adicionado + 2 conectores p/ alphasense * Falta expor ANx... * ESP32-C3 - ok * Dissipador onboard - Verificar * Regulador 3V3 * Um regulador para o esp32 e um para o rfm * ADD PMS5003 - ok"
- moved on the sheet: D8, J2, J3

Commit message: Add diversas trilhas e corrige 3dmodel
Parts:
- C34: footprint Capacitor_SMD:C_0805_2012Metric -> Capacitor_SMD:C_0603_1608Metric
- J14: footprint Connector_PinSocket_2.54mm:PinSocket_1x08_P2.54mm_Vertical_SMD_Pin1Left -> Connector_PinHeader_2.54mm:PinHeader_1x08_P2.54mm_Vertical
- R25, R26, R30, R31, R32, R33, R37: footprint Resistor_SMD:R_0805_2012Metric -> Resistor_SMD:R_0603_1608Metric
- U10: footprint Connector_JAE:JAE_LY20-16P-DLT1_2x08_P2.00mm_Horizontal -> RF_Module:HOPERF_RFM9XW_SMD
Changed lines of the file:
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@@
       (effects (font (size 1.27 1.27)) (justify left))
     )
-    (property "Footprint" "Resistor_SMD:R_0805_2012Metric" (at 342.392 35.56 90)
+    (property "Footprint" "Resistor_SMD:R_0603_1608Metric" (at 342.392 35.56 90)
       (effects (font (size 1.27 1.27)) hide)
     )
@@
       (effects (font (size 1.27 1.27)) (justify left))
     )
-    (property "Footprint" "Resistor_SMD:R_0805_2012Metric" (at 336.042 48.26 90)
+    (property "Footprint" "Resistor_SMD:R_0603_1608Metric" (at 336.042 48.26 90)
       (effects (font (size 1.27 1.27)) hide)
     )
@@
       (effects (font (size 1.27 1.27)) (justify left))
     )
-    (property "Footprint" "Capacitor_SMD:C_0805_2012Metric" (at 509.27 35.56 0)
+    (property "Footprint" "Capacitor_SMD:C_0603_1608Metric" (at 509.27 35.56 0)
       (effects (font (size 1.27 1.27)) hide)
     )
@@
       (effects (font (size 1.27 1.27)) (justify left))
     )
-    (property "Footprint" "Resistor_SMD:R_0805_2012Metric" (at 544.322 40.64 90)
+    (property "Footprint" "Resistor_SMD:R_0603_1608Metric" (at 544.322 40.64 90)
       (effects (font (size 1.27 1.27)) hide)
     )
@@
       (effects (font (size 1.27 1.27)) (justify left))
     )
-    (property "Footprint" "Resistor_SMD:R_0805_2012Metric" (at 408.432 82.55 90)
+    (property "Footprint" "Resistor_SMD:R_0603_1608Metric" (at 408.432 82.55 90)
       (effects (font (size 1.27 1.27)) hide)
     )
@@
       (effects (font (size 1.27 1.27)) (justify left))
     )
-    (property "Footprint" "Resistor_SMD:R_0805_2012Metric" (at 416.052 82.55 90)
+    (property "Footprint" "Resistor_SMD:R_0603_1608Metric" (at 416.052 82.55 90)
       (effects (font (size 1.27 1.27)) hide)
     )
@@
       (effects (font (size 1.27 1.27)) (justify left))
     )
-    (property "Footprint" "Resistor_SMD:R_0805_2012Metric" (at 402.082 82.55 90)
+    (property "Footprint" "Resistor_SMD:R_0603_1608Metric" (at 402.082 82.55 90)
       (effects (font (size 1.27 1.27)) hide)
     )
@@
       (effects (font (size 1.27 1.27)) (justify left))
     )
-    (property "Footprint" "Resistor_SMD:R_0805_2012Metric" (at 422.402 82.55 90)
+    (property "Footprint" "Resistor_SMD:R_0603_1608Metric" (at 422.402 82.55 90)
       (effects (font (size 1.27 1.27)) hide)
     )
@@
       (effects (font (size 1.27 1.27)) (justify left))
     )
-    (property "Footprint" "Connector_JAE:JAE_LY20-16P-DLT1_2x08_P2.00mm_Horizontal" (at 389.89 231.14 0)
+    (property "Footprint" "RF_Module:HOPERF_RFM9XW_SMD" (at 389.89 231.14 0)
       (effects (font (size 1.27 1.27)) hide)
     )
@@
       (effects (font (size 1.27 1.27)))
     )
-    (property "Footprint" "Connector_PinSocket_2.54mm:PinSocket_1x08_P2.54mm_Vertical_SMD_Pin1Left" (at 328.93 186.69 0)
+    (property "Footprint" "Connector_PinHeader_2.54mm:PinHeader_1x08_P2.54mm_Vertical" (at 328.93 186.69 0)
       (effects (font (size 1.27 1.27)) hide)
     )

Commit message: circuito esp32 ok
Parts:
- removed D10, D11: BAT54W, Package_TO_SOT_SMD:SOT-323_SC-70, symbol Diode:BAT54W
- added D11, D5: BAT54W, Diode_SMD:D_SOD-123, symbol Device:D_Schottky
- C29, C30, C31, C33: footprint Capacitor_SMD:C_0805_2012Metric -> Capacitor_SMD:C_0603_1608Metric
- R34: footprint Resistor_SMD:R_0805_2012Metric -> Resistor_SMD:R_0603_1608Metric
Connections:
- net +5V: now also D11.1 (K)
- net +9V: now also D5.1 (K)
- net BST_SW_5V: now also D11.2 (A)
- net BST_SW_9V: now also D5.2 (A)
- net ANT: now reaches AE1.1 (A), U10.9 (ANT)
Changed lines of the file:
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@@
     (effects (font (size 1.27 1.27)) (justify right bottom))
   )
+  (label "ANT" (at 492.76 265.43 0) (fields_autoplaced)
+    (effects (font (size 1.27 1.27)) (justify left bottom))
+  )
   (label "S2" (at 438.15 66.04 180) (fields_autoplaced)
     (effects (font (size 1.27 1.27)) (justify right bottom))
@@
     )
   )
-  (symbol (lib_id "Diode:BAT54W") (at 199.39 307.34 180) (unit 1)
-    (in_bom yes) (on_board yes) (dnp no)
-    (property "Reference" "D10" (at 199.39 301.625 0)
-      (effects (font (size 1.27 1.27)))
-    )
-    (property "Value" "BAT54W" (at 199.39 303.9364 0)
-      (effects (font (size 1.27 1.27)))
-    )
-    (property "Footprint" "Package_TO_SOT_SMD:SOT-323_SC-70" (at 199.39 302.895 0)
-      (effects (font (size 1.27 1.27)) hide)
-    )
-    (property "Datasheet" "https://assets.nexperia.com/documents/data-sheet/BAT54W_SER.pdf" (at 199.39 307.34 0)
-      (effects (font (size 1.27 1.27)) hide)
-    )
-    (pin "1")
-    (pin "2")
-    (pin "3")
-    (instances
-      (project "envcity_aqm_v2"
-        (path "/332e6a95-8453-45a7-bff6-50b465637d27"
-          (reference "D10") (unit 1)
-        )
-      )
-    )
-  )
   (symbol (lib_id "power:GND") (at 193.04 336.55 0) (unit 1)
     (in_bom yes) (on_board yes) (dnp no)
@@
     )
   )
-  (symbol (lib_id "Diode:BAT54W") (at 201.93 238.76 180) (unit 1)
-    (in_bom yes) (on_board yes) (dnp no)
-    (property "Reference" "D11" (at 201.93 233.045 0)
-      (effects (font (size 1.27 1.27)))
-    )
-    (property "Value" "BAT54W" (at 201.93 235.3564 0)
-      (effects (font (size 1.27 1.27)))
-    )
-    (property "Footprint" "Package_TO_SOT_SMD:SOT-323_SC-70" (at 201.93 234.315 0)
-      (effects (font (size 1.27 1.27)) hide)
-    )
-    (property "Datasheet" "https://assets.nexperia.com/documents/data-sheet/BAT54W_SER.pdf" (at 201.93 238.76 0)
-      (effects (font (size 1.27 1.27)) hide)
-    )
-    (pin "1")
-    (pin "2")
-    (pin "3")
-    (instances
-      (project "envcity_aqm_v2"
-        (path "/332e6a95-8453-45a7-bff6-50b465637d27"
-          (reference "D11") (unit 1)
-        )
-      )
-    )
-  )
   (symbol (lib_id "power:+9V") (at 247.65 234.95 0) (unit 1)
     (in_bom yes) (on_board yes) (dnp no)
@@
       (effects (font (size 1.27 1.27)) (justify left))
     )
-    (property "Footprint" "Capacitor_SMD:C_0805_2012Metric" (at 485.14 137.16 0)
+    (property "Footprint" "Capacitor_SMD:C_0603_1608Metric" (at 485.14 137.16 0)
       (effects (font (size 1.27 1.27)) hide)
     )
@@
       (effects (font (size 1.27 1.27)) (justify left))
     )
-    (property "Footprint" "Capacitor_SMD:C_0805_2012Metric" (at 439.42 160.02 0)
+    (property "Footprint" "Capacitor_SMD:C_0603_1608Metric" (at 439.42 160.02 0)
       (effects (font (size 1.27 1.27)) hide)
     )
@@
     )
   )
+  (symbol (lib_id "Device:D_Schottky") (at 199.39 307.34 180) (unit 1)
+    (in_bom yes) (on_board yes) (dnp no) (fields_autoplaced)
+    (property "Reference" "D11" (at 199.7075 303.0601 0)
+      (effects (font (size 1.27 1.27)))
+    )
+    (property "Value" "BAT54W" (at 199.7075 304.9811 0)
+      (effects (font (size 1.27 1.27)))
+    )
+    (property "Footprint" "Diode_SMD:D_SOD-123" (at 199.39 307.34 0)
+      (effects (font (size 1.27 1.27)) hide)
+    )
+    (property "Datasheet" "~" (at 199.39 307.34 0)
+      (effects (font (size 1.27 1.27)) hide)
+    )
+    (pin "1")
+    (pin "2")
+    (instances
+      (project "envcity_aqm_v2"
+        (path "/332e6a95-8453-45a7-bff6-50b465637d27"
+          (reference "D11") (unit 1)
+        )
+      )
+    )
+  )
   (symbol (lib_id "Device:R_Small") (at 464.82 129.54 0) (unit 1)
     (in_bom yes) (on_board yes) (dnp no)
@@
       (effects (font (size 1.27 1.27)) (justify left))
     )
-    (property "Footprint" "Resistor_SMD:R_0805_2012Metric" (at 464.82 129.54 0)
+    (property "Footprint" "Resistor_SMD:R_0603_1608Metric" (at 464.82 129.54 0)
       (effects (font (size 1.27 1.27)) hide)
     )
@@
     )
   )
+  (symbol (lib_id "Device:D_Schottky") (at 201.93 238.76 180) (unit 1)
+    (in_bom yes) (on_board yes) (dnp no) (fields_autoplaced)
+    (property "Reference" "D5" (at 202.2475 234.4801 0)
+      (effects (font (size 1.27 1.27)))
+    )
+    (property "Value" "BAT54W" (at 202.2475 236.4011 0)
+      (effects (font (size 1.27 1.27)))
+    )
+    (property "Footprint" "Diode_SMD:D_SOD-123" (at 201.93 238.76 0)
+      (effects (font (size 1.27 1.27)) hide)
+    )
+    (property "Datasheet" "~" (at 201.93 238.76 0)
+      (effects (font (size 1.27 1.27)) hide)
+    )
+    (pin "1")
+    (pin "2")
+    (instances
+      (project "envcity_aqm_v2"
+        (path "/332e6a95-8453-45a7-bff6-50b465637d27"
+          (reference "D5") (unit 1)
+        )
+      )
+    )
+  )
   (symbol (lib_id "power:GND") (at 426.72 161.29 0) (unit 1)
     (in_bom yes) (on_board yes) (dnp no) (fields_autoplaced)
@@
       (effects (font (size 1.27 1.27)) (justify left))
     )
-    (property "Footprint" "Capacitor_SMD:C_0805_2012Metric" (at 474.98 137.16 0)
+    (property "Footprint" "Capacitor_SMD:C_0603_1608Metric" (at 474.98 137.16 0)
       (effects (font (size 1.27 1.27)) hide)
     )
@@
       (effects (font (size 1.27 1.27)) (justify left))
     )
-    (property "Footprint" "Capacitor_SMD:C_0805_2012Metric" (at 464.82 137.16 0)
+    (property "Footprint" "Capacitor_SMD:C_0603_1608Metric" (at 464.82 137.16 0)
       (effects (font (size 1.27 1.27)) hide)
     )
