File: envcity_aqm_v2.kicad_sch (KiCad schematic)
At the start: 138 parts, among them IC1 DS1307ZN+, IC2 DMMT5401-7F, IC3 DMMT5401-7F, IC4 DMMT5401-7-F, IC6 ESP32-S2-SOLO-N4R2, J1 USB_B_Micro, J12 Conn_01x06_Male, J13 Conn_01x06_Male, J14 Conn_01x08_Pin, J15 Conn_01x02_Male, J16 Conn_01x02_Male, J2 Screw_Terminal_01x02, J3 Screw_Terminal_01x02, J4 MicroSD_Card MOLEX 5033981892, J5 Conn_01x03_Male, J6 Conn_01x04_Male, J7 Conn_01x06_Pin, J8 503398-1892, Q1 DMG2301L / DMP2045U, Q2 DMG2301L / DMP2045U, Q3 DMG2301L, Q4 DMG2301L, Q5 DMG2301L / DMP2045U, Q6 DMG2301L, Q7 DMN10H220L, Q8 DMN10H220L, SW1 BOOT, SW1 RESET, U1 TP4056, U10 RFM95W-915S2, U11 ADS1115IDGS, U2 USBLC6-2SC6, U3 MT3608, U4 MT3608, U5 LM2596S-5, U6 AP2112K-3.3, U7 DHT11, U8 AP2112K-3.3, U9 74HC4067DB, Y2 AB26TRB

Commit message: running DRC and fixing some errors
Parts:
- removed J4: MicroSD_Card MOLEX 5033981892, Connector_Card:microSD_HC_Hirose_DM3D-SF, symbol Connector:Micro_SD_Card
- R34, R37: footprint Resistor_SMD:R_0603_1608Metric -> Resistor_SMD:R_0402_1005Metric
Connections:
- net IO33 is gone; now on net ADS_ALERT: IC6.24 (IO33)
- net AIN0: now also J7.3 (Pin_3); no longer U9.1 (COM)
- net AIN1: now also U9.1 (COM); no longer J7.3 (Pin_3)
- net SD_CS: now also IC6.8 (IO15); no longer IC6.5 (IO5)
- net SD_MISO: now also IC6.5 (IO5); no longer IC6.8 (IO15)
- net SD_MOSI: now also IC6.7 (IO7); no longer IC6.6 (IO6)
- net SD_SCK: now also IC6.6 (IO6); no longer IC6.7 (IO7)
Changed lines of the file:
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@@
     (effects (font (size 1.27 1.27)) (justify left bottom))
   )
+  (label "ADS_ALERT" (at 457.2 210.82 180) (fields_autoplaced)
+    (effects (font (size 1.27 1.27)) (justify right bottom))
+  )
   (label "S0" (at 403.86 77.47 180) (fields_autoplaced)
     (effects (font (size 1.27 1.27)) (justify right bottom))
@@
     (effects (font (size 1.27 1.27)) (justify right bottom))
   )
-  (label "SD_SCK" (at 457.2 167.64 180) (fields_autoplaced)
+  (label "SD_SCK" (at 457.2 165.1 180) (fields_autoplaced)
     (effects (font (size 1.27 1.27)) (justify right bottom))
   )
@@
     (effects (font (size 0.9906 0.9906)) (justify left bottom))
   )
-  (label "AIN1" (at 297.18 313.69 0) (fields_autoplaced)
+  (label "AIN0" (at 297.18 313.69 0) (fields_autoplaced)
     (effects (font (size 1.27 1.27)) (justify left bottom))
   )
@@
     (effects (font (size 1.27 1.27)) (justify left bottom))
   )
-  (label "AIN0" (at 433.07 50.8 180) (fields_autoplaced)
+  (label "AIN1" (at 433.07 50.8 180) (fields_autoplaced)
     (effects (font (size 1.27 1.27)) (justify right bottom))
   )
@@
     (effects (font (size 1.27 1.27)) (justify right bottom))
   )
-  (label "SD_MOSI" (at 457.2 165.1 180) (fields_autoplaced)
+  (label "SD_MOSI" (at 457.2 167.64 180) (fields_autoplaced)
     (effects (font (size 1.27 1.27)) (justify right bottom))
   )
@@
     (effects (font (size 1.27 1.27)) (justify right bottom))
   )
-  (label "SD_MISO" (at 457.2 170.18 180) (fields_autoplaced)
+  (label "SD_MISO" (at 457.2 162.56 180) (fields_autoplaced)
     (effects (font (size 1.27 1.27)) (justify right bottom))
   )
@@
     (effects (font (size 1.27 1.27)) (justify right bottom))
   )
-  (label "IO33" (at 457.2 210.82 180) (fields_autoplaced)
-    (effects (font (size 1.27 1.27)) (justify right bottom))
-  )
   (label "SCL" (at 298.45 279.4 0) (fields_autoplaced)
     (effects (font (size 0.9906 0.9906)) (justify left bottom))
@@
     (effects (font (size 1.27 1.27)) (justify left bottom))
   )
-  (label "SD_CS" (at 457.2 162.56 180) (fields_autoplaced)
+  (label "SD_CS" (at 457.2 170.18 180) (fields_autoplaced)
     (effects (font (size 1.27 1.27)) (justify right bottom))
   )
@@
       (effects (font (size 1.27 1.27)) (justify left))
     )
-    (property "Footprint" "Resistor_SMD:R_0603_1608Metric" (at 544.322 40.64 90)
+    (property "Footprint" "Resistor_SMD:R_0402_1005Metric" (at 544.322 40.64 90)
       (effects (font (size 1.27 1.27)) hide)
     )
@@
     )
   )
-  (symbol (lib_id "Connector:Micro_SD_Card") (at -48.26 304.8 0) (unit 1)
-    (in_bom yes) (on_board yes) (dnp no)
-    (property "Reference" "J4" (at -49.53 286.5882 0)
-      (effects (font (size 1.27 1.27)))
-    )
-    (property "Value" "MicroSD_Card MOLEX 5033981892" (at -49.53 288.8996 0)
-      (effects (font (size 1.27 1.27)))
-    )
-    (property "Footprint" "Connector_Card:microSD_HC_Hirose_DM3D-SF" (at -19.05 297.18 0)
-      (effects (font (size 1.27 1.27)) hide)
-    )
-    (property "Datasheet" "http://katalog.we-online.de/em/datasheet/693072010801.pdf" (at -48.26 304.8 0)
-      (effects (font (size 1.27 1.27)) hide)
-    )
-    (property "LCSC Part#" "C428492" (at -48.26 304.8 0)
-      (effects (font (size 1.27 1.27)) hide)
-    )
-    (pin "1")
-    (pin "2")
-    (pin "3")
-    (pin "4")
-    (pin "5")
-    (pin "6")
-    (pin "7")
-    (pin "8")
-    (pin "9")
-    (instances
-      (project "envcity_aqm_v2"
-        (path "/332e6a95-8453-45a7-bff6-50b465637d27"
-          (reference "J4") (unit 1)
-        )
-      )
-    )
-  )
   (symbol (lib_id "Device:R_Small") (at 327.66 107.95 0) (unit 1)
     (in_bom yes) (on_board yes) (dnp no)
@@
       (effects (font (size 1.27 1.27)) (justify left))
     )
-    (property "Footprint" "Resistor_SMD:R_0603_1608Metric" (at 464.82 129.54 0)
+    (property "Footprint" "Resistor_SMD:R_0402_1005Metric" (at 464.82 129.54 0)
       (effects (font (size 1.27 1.27)) hide)
     )

Commit message: Corrigindo LCSC part #
Parts:
- removed C13, C9: 22uF-X5R, Capacitor_SMD:C_0805_2012Metric, symbol Device:C_Small
- removed D15: LED, LED_SMD:LED_0805_2012Metric_Pad1.15x1.40mm_HandSolder, symbol Device:LED
- removed D5: BAT54W, Diode_SMD:D_SOD-123, symbol Device:D_Schottky
- removed J5: Conn_01x03_Male, Connector_Molex:Molex_KK-254_AE-6410-03A_1x03_P2.54mm_Vertical, symbol envcity_aqm_v2-rescue:Conn_01x03_Male-Connector
- removed L2: XR0530-100M, Inductor_SMD:L_Chilisin_BMRA00050530, symbol Device:L_Small
- removed R13: 30K, Resistor_SMD:R_0603_1608Metric, symbol Device:R_Small_US
- removed R14: 2.2K, Resistor_SMD:R_0603_1608Metric, symbol Device:R_Small_US
- removed R18: 9K1, Resistor_SMD:R_0603_1608Metric, symbol Device:R
- removed U4: MT3608, Package_TO_SOT_SMD:SOT-23-6_Handsoldering, symbol envcity_aqm_v2-rescue:MT3608-MT3608
- C14: value 220uF-Tantalum -> 220uF-; JLCPCB Part# (none) -> C1954573
- IC1: JLCPCB Part # (none) -> C356706
- J1: footprint Connector_USB:USB_Micro-B_Wuerth_629105150521 -> Connector_USB:USB_Micro-B_Molex-105017-0001; JLCPCB Part # (none) -> C136000
- U11: JLCPCB Part# (none) -> C37593
- U3: JLCPCB Part # (none) -> C84817
- U5: JLCPCB Part # (none) -> C347421
- U9: LCSC Part# C124924 -> C98457
Connections:
- net S0: now also IC6.38 (IO2); no longer IC6.39 (IO1)
- net S1: now also IC6.39 (IO1); no longer IC6.38 (IO2)
Other:
- note removed: "* The GND pin located in the middle provides an easy path for the return current for both the 9V and anem_analog circuits."
- note removed: "Anemômetro"
- note removed: "Conversor Step-Up 9V"
- note removed: "LED - StepUp 9V"
