File: envcity_aqm_v2.kicad_sch (KiCad schematic)
At the start: 134 parts, among them IC1 DS1307ZN+, IC2 DMMT5401-7F, IC3 DMMT5401-7F, IC4 DMMT5401-7-F, IC6 ESP32-S2-SOLO-N4R2, J1 USB_B_Micro, J12 Conn_01x06_Male, J13 Conn_01x06_Male, J14 Conn_01x08_Pin, J15 Conn_01x02_Male, J16 Conn_01x02_Male, J2 Screw_Terminal_01x02, J3 Screw_Terminal_01x02, J6 Conn_01x04_Male, J7 Conn_01x06_Pin, J8 503398-1892, Q1 DMP2045U-7, Q2 DMP2045U-7, Q3 DMP2045U-7, Q4 DMP2045U-7, Q5 DMP2045U-7, Q6 DMP2045U-7, Q7 DMN10H220L, Q8 DMN10H220L, SW1 BOOT, SW1 RESET, U1 TP4056, U10 RFM95W-915, U11 ADS1115IDGS, U12 TPS54202DDC, U2 USBLC6-2SC6, U3 MT3608, U4 SHT30-DIS, U6 AP2112K-3.3, U7 DHT11, U8 AP2112K-3.3, U9 74HC4067DB, Y2 FC-135R

Commit message: Add logo na pcb
Add a logo
Parts:
- BT1: LCSC Part # (none) -> C70377; LCSC Part# C70377 -> (none)
- C11, C15, C22, C23: LCSC C19702 -> (none); LCSC Part # (none) -> C19702
- C16, C24: LCSC C14663 -> (none); LCSC Part # (none) -> C14663
- D16, D7: LCSC C2289 -> (none); LCSC Part # (none) -> C2289
- EQ3: LCSC # C504992 -> (none); LCSC Part # (none) -> C504992
- IC6: LCSC Part # (none) -> C3040594; LCSC Part# C3040594 -> (none)
- J8: LCSC Part # (none) -> C428492; LCSC Part# C428492 -> (none)
- L1: LCSC Part # (none) -> C5307602; LCSC Part# C5307602 -> (none)
- L2: LCSC Part # (none) -> C189932; LCSC Part# C189932 -> (none)
- Q1, Q2, Q3, Q4, Q5, Q6: LCSC Part # (none) -> C459541; LCSC Part# C459541 -> (none)
- R10, R22, R23, R8: LCSC C25804 -> (none); LCSC Part # (none) -> C25804
- SW1: JLCPCB Part # (none) -> C221897; JLCPCB Part#  C221897 -> (none)
- SW1: JLCPCB Part # (none) -> C221897; JLCPCB Part# C221897 -> (none)
- U10: LCSC # C2844473 -> (none); LCSC Part # (none) -> C2844473
- U11: JLCPCB Part # (none) -> C37593; JLCPCB Part# C37593 -> (none)
- U4: LCSC Part # (none) -> C2687423; LCSC Part# C2687423 -> (none)
- U6, U8: LCSC Part # (none) -> C51118; LCSC Part# C51118 -> (none)
- U9: LCSC Part # (none) -> C98457; LCSC Part# C98457 -> (none)
Changed lines of the file:
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@@
       (effects (font (size 1.27 1.27)) hide)
     )
-    (property "LCSC Part#" "C5307602" (at 176.53 248.92 90)
+    (property "LCSC Part #" "C5307602" (at 176.53 248.92 0)
       (effects (font (size 1.27 1.27)) hide)
     )
@@
       (effects (font (size 1.27 1.27)) hide)
     )
-    (property "JLCPCB Part#" "C37593" (at 520.7 53.34 0)
+    (property "JLCPCB Part #" "C37593" (at 520.7 53.34 0)
       (effects (font (size 1.27 1.27)) hide)
     )
@@
       (effects (font (size 1.27 1.27)) hide)
     )
-    (property "LCSC Part#" "C98457" (at 452.12 63.5 0)
+    (property "LCSC Part #" "C98457" (at 452.12 63.5 0)
       (effects (font (size 1.27 1.27)) hide)
     )
@@
       (effects (font (size 1.27 1.27)) hide)
     )
-    (property "LCSC #" "C504992" (at 325.12 252.73 0)
+    (property "LCSC Part #" "C504992" (at 325.12 252.73 0)
       (effects (font (size 1.27 1.27)) hide)
     )
@@
       (effects (font (size 1.27 1.27)) (justify left) hide)
     )
-    (property "LCSC Part#" "C459541" (at 337.82 59.69 90)
+    (property "LCSC Part #" "C459541" (at 337.82 59.69 0)
       (effects (font (size 1.27 1.27)) hide)
     )
@@
       (effects (font (size 1.27 1.27)) (justify left) hide)
     )
-    (property "LCSC Part#" "C459541" (at 107.95 133.35 90)
+    (property "LCSC Part #" "C459541" (at 107.95 133.35 0)
       (effects (font (size 1.27 1.27)) hide)
     )
@@
       (effects (font (size 1.27 1.27)) hide)
     )
-    (property "LCSC Part#" "C70377" (at 38.1 295.91 0)
+    (property "LCSC Part #" "C70377" (at 38.1 295.91 0)
       (effects (font (size 1.27 1.27)) hide)
     )
@@
       (effects (font (size 1.27 1.27)) (justify left) hide)
     )
-    (property "LCSC Part#" "C459541" (at 242.57 40.64 90)
+    (property "LCSC Part #" "C459541" (at 242.57 40.64 0)
       (effects (font (size 1.27 1.27)) hide)
     )
@@
       (effects (font (size 1.27 1.27)) (justify left) hide)
     )
-    (property "LCSC Part#" "C459541" (at 288.29 49.53 90)
+    (property "LCSC Part #" "C459541" (at 288.29 49.53 0)
       (effects (font (size 1.27 1.27)) hide)
     )
@@
       (effects (font (size 1.27 1.27)) (justify left) hide)
     )
-    (property "LCSC Part#" "C459541" (at 341.63 83.82 90)
+    (property "LCSC Part #" "C459541" (at 341.63 83.82 0)
       (effects (font (size 1.27 1.27)) hide)
     )
@@
       (effects (font (size 1.27 1.27)) (justify left) hide)
     )
-    (property "LCSC Part#" "C459541" (at 107.95 85.09 90)
+    (property "LCSC Part #" "C459541" (at 107.95 85.09 0)
       (effects (font (size 1.27 1.27)) hide)
     )
@@
       (effects (font (size 1.27 1.27)) (justify left) hide)
     )
-    (property "LCSC Part#" "C428492" (at 53.34 341.63 0)
+    (property "JLCPCB Part #" "C428492" (at 53.34 341.63 0)
       (effects (font (size 1.27 1.27)) hide)
     )
-    (property "JLCPCB Part #" "C428492" (at 53.34 341.63 0)
+    (property "LCSC Part #" "C428492" (at 53.34 341.63 0)
       (effects (font (size 1.27 1.27)) hide)
     )
@@
       (effects (font (size 1.27 1.27)) hide)
     )
-    (property "LCSC" "C25804" (at 171.45 378.46 0)
+    (property "LCSC Part #" "C25804" (at 171.45 378.46 0)
       (effects (font (size 1.27 1.27)) hide)
     )
@@
       (effects (font (size 1.27 1.27)) hide)
     )
-    (property "LCSC Part#" "C51118" (at 199.39 316.23 0)
+    (property "LCSC Part #" "C51118" (at 199.39 316.23 0)
       (effects (font (size 1.27 1.27)) hide)
     )
@@
       (effects (font (size 1.27 1.27)) hide)
     )
-    (property "LCSC" "C2289" (at 171.45 388.62 90)
+    (property "LCSC Part #" "C2289" (at 171.45 388.62 0)
       (effects (font (size 1.27 1.27)) hide)
     )
@@
       (effects (font (size 1.27 1.27)) hide)
     )
-    (property "LCSC Part#" "C2687423" (at 292.1 232.41 0)
+    (property "JLCPCB Part #" "C2687423" (at 292.1 232.41 0)
       (effects (font (size 1.27 1.27)) hide)
     )
-    (property "JLCPCB Part #" "C2687423" (at 292.1 232.41 0)
+    (property "LCSC Part #" "C2687423" (at 292.1 232.41 0)
       (effects (font (size 1.27 1.27)) hide)
     )
@@
       (effects (font (size 1.27 1.27)) hide)
     )
-    (property "LCSC" "C25804" (at 186.69 374.65 0)
+    (property "LCSC Part #" "C25804" (at 186.69 374.65 0)
       (effects (font (size 1.27 1.27)) hide)
     )
@@
       (effects (font (size 1.27 1.27)) hide)
     )
-    (property "LCSC" "C2289" (at 170.18 330.2 90)
+    (property "LCSC Part #" "C2289" (at 170.18 330.2 0)
       (effects (font (size 1.27 1.27)) hide)
     )
@@
       (effects (font (size 1.27 1.27)) hide)
     )
-    (property "LCSC Part#" "C189932" (at 204.47 182.88 90)
+    (property "LCSC Part #" "C189932" (at 204.47 182.88 0)
       (effects (font (size 1.27 1.27)) hide)
     )
@@
       (effects (font (size 1.27 1.27)) hide)
     )
-    (property "LCSC #" "C2844473" (at 473.71 273.05 0)
+    (property "AlternativeValue" "DreamLNK DL-RFM95-915M" (at 473.71 273.05 0)
       (effects (font (size 1.27 1.27)) hide)
     )
-    (property "AlternativeValue" "DreamLNK DL-RFM95-915M" (at 473.71 273.05 0)
+    (property "LCSC Part #" "C2844473" (at 473.71 273.05 0)
       (effects (font (size 1.27 1.27)) hide)
     )
@@
       (effects (font (size 1.27 1.27)) hide)
     )
-    (property "LCSC" "C19702" (at 222.25 318.77 0)
+    (property "LCSC Part #" "C19702" (at 222.25 318.77 0)
       (effects (font (size 1.27 1.27)) hide)
     )
@@
       (effects (font (size 1.27 1.27)) hide)
     )
-    (property "LCSC" "C19702" (at 213.36 377.19 0)
+    (property "LCSC Part #" "C19702" (at 213.36 377.19 0)
       (effects (font (size 1.27 1.27)) hide)
     )
@@
       (effects (font (size 1.27 1.27)) hide)
     )
-    (property "LCSC" "C19702" (at 223.52 377.19 0)
+    (property "LCSC Part #" "C19702" (at 223.52 377.19 0)
       (effects (font (size 1.27 1.27)) hide)
     )
@@
       (effects (font (size 1.27 1.27)) hide)
     )
-    (property "LCSC" "C14663" (at 233.68 377.19 0)
+    (property "LCSC Part #" "C14663" (at 233.68 377.19 0)
       (effects (font (size 1.27 1.27)) hide)
     )
@@
       (effects (font (size 1.27 1.27)) (justify left top) hide)
     )
-    (property "LCSC Part#" "C3040594" (at 462.28 152.4 0)
+    (property "LCSC Part #" "C3040594" (at 462.28 152.4 0)
       (effects (font (size 1.27 1.27)) hide)
     )
@@
       (effects (font (size 1.27 1.27)) hide)
     )
-    (property "LCSC" "C25804" (at 170.18 320.04 0)
+    (property "LCSC Part #" "C25804" (at 170.18 320.04 0)
       (effects (font (size 1.27 1.27)) hide)
     )
@@
       (effects (font (size 1.27 1.27)) hide)
     )
-    (property "LCSC" "C19702" (at 212.09 318.77 0)
+    (property "LCSC Part #" "C19702" (at 212.09 318.77 0)
       (effects (font (size 1.27 1.27)) hide)
     )
@@
       (effects (font (size 1.27 1.27)) hide)
     )
-    (property "LCSC" "C14663" (at 232.41 318.77 0)
+    (property "LCSC Part #" "C14663" (at 232.41 318.77 0)
       (effects (font (size 1.27 1.27)) hide)
     )
@@
       (effects (font (size 1.27 1.27)) hide)
     )
-    (property "JLCPCB Part# " "C221897" (at 506.73 144.78 0)
+    (property "JLCPCB Part #" "C221897" (at 506.73 144.78 0)
       (effects (font (size 1.27 1.27)) hide)
     )
@@
       (effects (font (size 1.27 1.27)) hide)
     )
-    (property "LCSC" "C25804" (at 185.42 316.23 0)
+    (property "LCSC Part #" "C25804" (at 185.42 316.23 0)
       (effects (font (size 1.27 1.27)) hide)
     )
@@
       (effects (font (size 1.27 1.27)) hide)
     )
-    (property "LCSC Part#" "C51118" (at 200.66 374.65 0)
+    (property "LCSC Part #" "C51118" (at 200.66 374.65 0)
       (effects (font (size 1.27 1.27)) hide)
     )
@@
       (effects (font (size 1.27 1.27)) hide)
     )
-    (property "JLCPCB Part#" "C221897" (at 439.42 154.94 0)
+    (property "JLCPCB Part #" "C221897" (at 439.42 154.94 0)
       (effects (font (size 1.27 1.27)) hide)
     )

Commit message: add novo esp32
Parts:
- removed D16, D7: LED, LED_SMD:LED_0603_1608Metric, symbol Device:LED
- removed IC6: ESP32-S2-SOLO-N4R2, ESP32-S2-SOLO-N4R2:ESP32S2SOLON4R2, symbol ESP32-S2-SOLO-N4R2:ESP32-S2-SOLO-N4R2
- removed R22: 10k, Resistor_SMD:R_0805_2012Metric, symbol Device:R_US
- removed R8: 10k, Resistor_SMD:R_0603_1608Metric, symbol Device:R_US
- added IC5: ESP32-S3-WROOM-1-N16, ESP32-S3:ESP32S3WROOM1N16, symbol ESP32-S3-WROOM-1-N16:ESP32-S3-WROOM-1-N16
- C1, C28: LCSC Part # (none) -> C19702
- C17, C18, C19, C2, C20, C21, C25, C26, C27, C29, C32, C33, C34, C35, C36, C4, C9: LCSC Part # (none) -> C14663
- D11: LCSC Part # (none) -> C915628
- D2: footprint Diode_SMD:D_SOD-523 -> AB26TRB-32.768KHZ-T:PESD24VS1ULQZ; LCSC Part # C1974922 -> C2844735
- EQ1, EQ2, EQ4, J12, J13: LCSC Part # (none) -> C2847672
- EQ3: LCSC Part # C504992 -> C2847672
- IC1: LCSC Part # (none) -> C356706
- IC4: value DMMT5401-7-F -> DMMT5401-7F
- J1: LCSC Part # (none) -> C136000
- J14: LCSC Part # (none) -> C240845
- J15: LCSC Part # C505162 -> C509147
- J16: LCSC Part # (none) -> C509147
- J3: LCSC Part # (none) -> C3029316
- Q7, Q8: LCSC Part # (none) -> C5122013
- R15, R20, R24, R25, R26: LCSC Part # (none) -> C25804
- R16, R17, R2, R3, R35, R36: LCSC Part # (none) -> C23162
- R18, R38: footprint Capacitor_SMD:C_0603_1608Metric_Pad1.08x0.95mm_HandSolder -> Resistor_SMD:R_0603_1608Metric
- R28, R29, R34, R4, R5: LCSC Part # (none) -> C25744
- R30, R31, R32, R33: footprint Resistor_SMD:R_0402_1005Metric_Pad0.72x0.64mm_HandSolder -> Resistor_SMD:R_0402_1005Metric; LCSC Part # (none) -> C25900
- R37: LCSC Part # (none) -> C25900
- SW1: LCSC Part # (none) -> C221897
- U1: LCSC Part # (none) -> C382139
- U11: LCSC Part # (none) -> C37593
- U3: LCSC Part # (none) -> C84817
- U7: value DHT11 -> DHT22
- U9: LCSC Part # C98457 -> C97702
- Y2: JLCPCB Part # C1987155 -> C94276; LCSC Part # C179645 -> C94276
Connections:
- net +3V3: now also IC5.2 (3V3)
- net ADS_ALERT: now also IC5.24 (IO47)
- net BOOT: now also IC5.27 (IO0)
- net DHT_PIN: now also IC5.23 (IO21)
- net EN: now also IC5.3 (EN)
- net ESP_USB_D+: now also IC5.14 (IO20)
- net ESP_USB_D-: now also IC5.13 (IO19)
- net FAN1: now also IC5.9 (IO16); no longer Q7.1 (G)
- net FAN2: now also Q7.1 (G), IC5.17 (IO9)
- net GND: now also IC5.1 (GND_1), IC5.40 (GND_2), IC5.41 (GND_3), IC5.42 (GND_4), IC5.43 (GND_5), IC5.44 (GND_6), IC5.45 (GND_7), IC5.46 (GND_8), IC5.47 (GND_9), IC5.48 (GND_10), IC5.49 (GND_11)
- net IO12: now also IC5.20 (IO12)
- net IO13: now also IC5.21 (IO13)
- net IO8: now also IC5.12 (IO8)
- net PMS_RX: now also IC5.28 (IO35)
- net PMS_TX: now also IC5.25 (IO48)
- net RFM_CS: now also IC5.29 (IO36)
- net RFM_DIO0: now also IC5.33 (IO40)
- net RFM_DIO1: now also IC5.34 (IO41)
- net RFM_DIO2: now also IC5.35 (IO42)
- net RFM_MISO: now also IC5.30 (IO37)
- net RFM_MOSI: now also IC5.31 (IO38)
- net RFM_RST: now also IC5.22 (IO14)
- net RFM_SCK: now also IC5.32 (IO39)
- net S0: now also IC5.38 (IO2)
- net S1: now also IC5.39 (IO1)
- net S2: now also IC5.10 (IO17)
- net S3: now also IC5.11 (IO18)
- net SCL: now also IC5.19 (IO11)
- net SDA: now also IC5.18 (IO10)
- net SD_CS: now also IC5.8 (IO15)
- net SD_MISO: now also IC5.5 (IO5)
- net SD_MOSI: now also IC5.7 (IO7)
- net SD_SCK: now also IC5.6 (IO6)
- no-connect marks 21 -> 22

Commit message: add sim
Connections:
- net Vusb: no longer IC2.2 (B), IC2.3 (B)
- net at IC2.1 (C), R15.1: now also IC2.2 (B), IC2.3 (B)
Changed lines of the file:
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@@
   (junction (at 161.29 180.34) (diameter 0) (color 0 0 0 0)
   )
+  (junction (at 238.76 53.34) (diameter 0) (color 0 0 0 0)
+  )
   (junction (at 223.52 372.11) (diameter 0) (color 0 0 0 0)
   )
@@
   (junction (at 213.36 372.11) (diameter 0) (color 0 0 0 0)
   )
-  (junction (at 228.6 44.45) (diameter 0) (color 0 0 0 0)
-  )
   (junction (at 274.32 53.34) (diameter 0) (color 0 0 0 0)
   )
@@
   (junction (at 337.82 222.25) (diameter 0) (color 0 0 0 0)
   )
-  (junction (at 238.76 53.34) (diameter 0) (color 0 0 0 0)
-  )
   (junction (at 364.49 222.25) (diameter 0) (color 0 0 0 0)
   )
@@
   )
   (junction (at 290.83 177.8) (diameter 0) (color 0 0 0 0)
+  )
+  (junction (at 228.6 59.69) (diameter 0) (color 0 0 0 0)
   )
   (no_connect (at 96.52 351.79))
@@
     (stroke (width 0) (type default))
   )
-  (wire (pts (xy 228.6 48.26) (xy 228.6 44.45))
+  (wire (pts (xy 228.6 38.1) (xy 228.6 48.26))
     (stroke (width 0) (type default))
   )
@@
     (stroke (width 0) (type default))
   )
+  (wire (pts (xy 238.76 59.69) (xy 228.6 59.69))
+    (stroke (width 0) (type default))
+  )
   (polyline (pts (xy 313.69 261.62) (xy 274.32 261.62))
     (stroke (width 0) (type default))
@@
     (stroke (width 0) (type default))
   )
-  (wire (pts (xy 228.6 38.1) (xy 228.6 44.45))
-    (stroke (width 0) (type default))
-  )
   (wire (pts (xy 85.09 290.83) (xy 90.17 290.83))
     (stroke (width 0) (type default))
@@
     (stroke (width 0) (type default))
   )
-  (wire (pts (xy 228.6 58.42) (xy 228.6 62.23))
+  (wire (pts (xy 228.6 58.42) (xy 228.6 59.69))
     (stroke (width 0) (type default))
   )
@@
     (stroke (width 0) (type default))
   )
-  (wire (pts (xy 241.3 53.34) (xy 238.76 53.34))
+  (wire (pts (xy 236.22 53.34) (xy 238.76 53.34))
     (stroke (width 0) (type default))
   )
@@
     (stroke (width 0) (type default))
   )
+  (wire (pts (xy 238.76 53.34) (xy 241.3 53.34))
+    (stroke (width 0) (type default))
+  )
   (wire (pts (xy 115.57 40.64) (xy 115.57 41.91))
     (stroke (width 0) (type default))
@@
     (stroke (width 0) (type default))
   )
+  (wire (pts (xy 228.6 59.69) (xy 228.6 62.23))
+    (stroke (width 0) (type default))
+  )
   (bus (pts (xy 420.37 73.66) (xy 426.72 73.66))
     (stroke (width 0) (type default))
@@
     (stroke (width 0) (type default))
   )
+  (wire (pts (xy 238.76 53.34) (xy 238.76 59.69))
+    (stroke (width 0) (type default))
+  )
   (wire (pts (xy 33.02 349.25) (xy 53.34 349.25))
     (stroke (width 0) (type default))
@@
     (stroke (width 0) (type default))
   )
-  (wire (pts (xy 238.76 53.34) (xy 236.22 53.34))
-    (stroke (width 0) (type default))
-  )
   (wire (pts (xy 361.95 234.95) (xy 361.95 236.22))
     (stroke (width 0) (type default))
@@
     (stroke (width 0) (type default))
   )
-  (wire (pts (xy 228.6 44.45) (xy 238.76 44.45))
-    (stroke (width 0) (type default))
-  )
   (wire (pts (xy 180.34 24.13) (xy 180.34 27.94))
     (stroke (width 0) (type default))
@@
     (stroke (width 0) (type default))
   )
-  (wire (pts (xy 238.76 44.45) (xy 238.76 53.34))
-    (stroke (width 0) (type default))
-  )

Commit message: add flyback diode. add pulldown on fan switch fet
Parts:
- added D5, D6: SS14, Diode_SMD:D_SMA, symbol Diode:SS14
- added R22, R40: 10k, Resistor_SMD:R_0805_2012Metric, symbol Device:R_Small
- added R39, R8: 1k, Resistor_SMD:R_0805_2012Metric, symbol Device:R_Small
- AE1: symbol Device:Antenna -> Device:Antenna_Shield
- renumbered SW1 to SW2
Connections:
- net +5V: now also D5.1 (K), D6.1 (K)
- net FAN1: now also R39.1
- net FAN2: now also R8.1; no longer Q7.1 (G), Q8.1 (G)
- net GND: now also AE1.2 (Shield), R22.1, R40.1
- net Vexternal: no longer IC4.2 (B), IC4.3 (B)
- net Vsolar_reg: no longer IC3.2 (B), IC3.3 (B)
- net at J15.2 (Pin_2), Q7.3 (D): now also D6.2 (A)
- net at IC3.1 (C), R20.1: now also IC3.2 (B), IC3.3 (B)
- net at IC4.1 (C), R24.1: now also IC4.2 (B), IC4.3 (B)
- net at J16.2 (Pin_2), Q8.3 (D): now also D5.2 (A)
- new net: Q7.1 (G), R39.2, R40.2
- new net: Q8.1 (G), R22.2, R8.2
- no-connect marks 22 -> 26
Other:
- moved on the sheet: Q8
