File: envcity_aqm_v2.kicad_pcb (KiCad board)
At the start: 2 copper layers, 100 x 100 mm, 136 parts, among them IC1 DS1307ZN+, IC2 DMMT5401-7F, IC3 DMMT5401-7F, IC4 DMMT5401-7-F, IC6 ESP32-S2-SOLO-N4R2, J1 USB_B_Micro, J10 Conn_01x06_Male, J11 Conn_01x06_Male, J12 Conn_01x06_Male, J13 Conn_01x06_Male, J14 Conn_01x08_Pin, J15 Conn_01x02_Male, J16 Conn_01x02_Male, J2 Screw_Terminal_01x02, J3 Screw_Terminal_01x02, J4 Micro_SD_Card, J5 Conn_01x03_Male, J6 Conn_01x04_Male, J7 Conn_01x06_Pin, J8 Conn_01x06_Male, J9 Conn_01x06_Male, Q1 DMG2301L / DMP2045U, Q2 DMG2301L / DMP2045U, Q3 DMG2301L, Q4 DMG2301L, Q5 DMG2301L / DMP2045U, Q6 DMG2301L, Q7 DMN10H220L, Q8 DMN10H220L, SW1 RESET, SW2 BOOT, U1 TP4056, U10 RFM95W-915S2, U11 ADS1115IDGS, U2 USBLC6-2SC6, U3 MT3608, U4 MT3608, U5 LM2596S-5, U6 AP2112K-3.3, U7 DHT11, U8 AP2112K-3.3, U9 74HC4067DB, Y2 AB26TRB

Commit message: Terminando o posicionamento dos components
Parts:
- added C35: 100nF, Capacitor_SMD:C_0603_1608Metric, F.Cu at (198.1, 120.8)
- C18, C19, C20, C21, C25, C26, C27: footprint Capacitor_SMD:C_0805_2012Metric -> Capacitor_SMD:C_0603_1608Metric
- J14: footprint Connector_PinHeader_2.54mm:PinHeader_1x08_P2.54mm_Vertical -> Connector_Molex:Molex_PicoBlade_53047-0810_1x08_P1.25mm_Vertical
- J7: footprint Connector_Molex:Molex_KK-254_AE-6410-06A_1x06_P2.54mm_Vertical -> Connector_PinHeader_2.54mm:PinHeader_1x06_P2.54mm_Vertical
- moved H1 323.4 mm to (234.2, 136.8)
- moved H2 323.4 mm to (234.2, 143.4)
- moved H3 323.4 mm to (234.2, 149.9)
- moved H4 323.4 mm to (234.2, 156.5)
- moved C22 137.2 mm to (190.9, 67.6)
- moved C23 137.2 mm to (188.4, 67.6)
- moved D16 137.2 mm to (177.4, 65.7)
- moved R22 137.2 mm to (180.4, 65.7)
- moved R23 137.2 mm to (179.4, 69.7)
- moved U8 137.2 mm to (184.4, 67.7)
- moved C24 137.2 mm to (184.3, 63.6)
- moved U7 122.0 mm to (186.2, 86.5), turned to -90 degrees
- moved R28 118.3 mm to (229.6, 93.1)
- moved R29 114.7 mm to (229.5, 89.8)
- moved C9 113.8 mm to (167.1, 124.2), turned to -90 degrees
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- renumbered J8 to EQ1, J9 to EQ2, J10 to EQ3, J11 to EQ4
Connections:
- IC6 pad 17: unconnected-(IC6-IO9-Pad17) -> /RFM_CS
- IC6 pad 18: /RFM_CS -> /RFM_SCK
- IC6 pad 21: /RFM_SCK -> unconnected-(IC6-IO13-Pad21)
- IC6 pad 23: /RFM_DIO0 -> /RFM_DIO2
- IC6 pad 25: /RFM_DIO2 -> /RFM_DIO0
- J5 pad 3: /I7 -> /I12
Routing:
- net +5V: track 42.5 -> 314.7 mm, vias 0 -> 13
- net /RFM_CS: track 0.00 -> 58.9 mm
- net /I7: track 0.00 -> 57.1 mm
- net /RFM_SCK: track 0.00 -> 54.0 mm
- net /RFM_RST: track 0.00 -> 51.4 mm
- net /PMS_TX: track 0.00 -> 50.6 mm, vias 0 -> 4
- net /PMS_RX: track 0.00 -> 50.3 mm, vias 0 -> 4
- net /I6: track 0.00 -> 49.1 mm
- net /RFM_MOSI: track 0.00 -> 48.8 mm
- net /RFM_MISO: track 0.00 -> 42.6 mm
- net /RFM_DIO0: track 0.00 -> 42.6 mm, vias 0 -> 2
- net /RFM_DIO1: track 0.00 -> 41.9 mm, vias 0 -> 2
- net Vsys: track 8.55 -> 49.8 mm, vias 0 -> 4
- net /RFM_DIO2: track 0.00 -> 41.2 mm, vias 0 -> 2
- net /I9: track 0.00 -> 39.9 mm, vias 0 -> 2
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- added copper zone on F.Cu, net /BST_SW_9V
- added copper zone on F.Cu, net /Vsolar
- added copper zone on F.Cu, net Vexternal
- added copper zone on B.Cu, net Vusb
- removed copper zone on B.Cu, net Vexternal
Other:
- board text added: "5V"

Commit message: mudando posicoes
Parts:
- moved R33 9.00 mm to (192.2, 135.3), turned to 45 degrees
- moved R32 8.68 mm to (191.0, 134.0), turned to 45 degrees
- moved C28 8.02 mm to (186.9, 130.4), turned to 45 degrees
- moved R30 6.96 mm to (187.8, 146.4), turned to 45 degrees
- moved R35 5.45 mm to (175.8, 76.1), turned to -90 degrees
- moved R31 5.21 mm to (186.2, 144.8), turned to 45 degrees
- moved U9 2.11 mm to (184.2, 138.2), turned to 45 degrees
- moved C34 0.65 mm to (171.5, 136.8)
Connections:
- IC6 pad 28: unconnected-(IC6-IO35-Pad28) -> /DHT_PIN
- IC6 pad 35: /DHT_PIN -> unconnected-(IC6-IO42-Pad35)
Routing:
- net /I7: track 57.1 -> 0.00 mm
- net /I6: track 49.1 -> 0.00 mm
- net /I5: track 38.0 -> 0.00 mm
- net /I8: track 35.4 -> 0.00 mm
- net /I4: track 34.8 -> 0.00 mm
- net /I11: track 29.6 -> 0.00 mm, vias 1 -> 0
- net /I10: track 28.7 -> 0.00 mm
- net /I9: track 39.9 -> 18.1 mm
- net /I3: track 20.4 -> 0.00 mm
- net /I0: track 19.3 -> 0.00 mm
- net /I2: track 18.6 -> 0.00 mm
- net /I1: track 17.4 -> 0.00 mm
- net /S0: track 10.0 -> 0.00 mm
- net /DHT_PIN: track 21.4 -> 15.4 mm
- net /S1: track 5.88 -> 0.00 mm
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