File: sensors/sensors.sch (KiCad schematic (older format))
At the start: 8 parts, among them J10 Conn_01x06_Male, J11 Conn_01x06_Male, J12 Conn_01x03_Female, J6 Conn_01x06_Male, J7 Conn_01x06_Male, J8 Conn_01x06_Male, J9 Conn_01x06_Male, U7 DHT11

Commit message: v3
Parts:
- renumbered J11 to J10, J12 to J11, J6 to J5, J7 to J6, J8 to J7, J9 to J8, J10 to J9, U7 to U8
Changed lines of the file:
@@
 $Descr A4 11693 8268
 encoding utf-8
-Sheet 7 7
+Sheet 6 7
 Title ""
 Date "2021-12-26"
@@
 	2750 850  2750 2400
 $Comp
-L Connector:Conn_01x06_Male J9
+L Connector:Conn_01x06_Male J8
 U 1 1 61C57284
 P 2850 1600
-F 0 "J9" H 3100 2000 50  0000 C CNN
+F 0 "J8" H 3100 2000 50  0000 C CNN
 F 1 "Conn_01x06_Male" H 3100 1900 50  0000 C CNN
 F 2 "Connector_Molex:Molex_KK-254_AE-6410-06A_1x06_P2.54mm_Vertical" H 2850 1600 50  0001 C CNN
@@
 	1350 2900 1350 4450
 $Comp
-L Connector:Conn_01x06_Male J7
+L Connector:Conn_01x06_Male J6
 U 1 1 61C5F8EA
 P 1450 3650
-F 0 "J7" H 1700 4050 50  0000 C CNN
+F 0 "J6" H 1700 4050 50  0000 C CNN
 F 1 "Conn_01x06_Male" H 1700 3950 50  0000 C CNN
 F 2 "Connector_Molex:Molex_KK-254_AE-6410-06A_1x06_P2.54mm_Vertical" H 1450 3650 50  0001 C CNN
@@
 	2750 2900 2750 4450
 $Comp
-L Connector:Conn_01x06_Male J10
+L Connector:Conn_01x06_Male J9
 U 1 1 61C5F904
 P 2850 3650
-F 0 "J10" H 3100 4050 50  0000 C CNN
+F 0 "J9" H 3100 4050 50  0000 C CNN
 F 1 "Conn_01x06_Male" H 3100 3950 50  0000 C CNN
 F 2 "Connector_Molex:Molex_KK-254_AE-6410-06A_1x06_P2.54mm_Vertical" H 2850 3650 50  0001 C CNN
@@
 	1350 4850 1350 6400
 $Comp
-L Connector:Conn_01x06_Male J8
+L Connector:Conn_01x06_Male J7
 U 1 1 61C64616
 P 1450 5600
-F 0 "J8" H 1700 6000 50  0000 C CNN
+F 0 "J7" H 1700 6000 50  0000 C CNN
 F 1 "Conn_01x06_Male" H 1700 5900 50  0000 C CNN
 F 2 "Connector_Molex:Molex_KK-254_AE-6410-06A_1x06_P2.54mm_Vertical" H 1450 5600 50  0001 C CNN
@@
 	2750 4850 2750 6400
 $Comp
-L Connector:Conn_01x06_Male J11
+L Connector:Conn_01x06_Male J10
 U 1 1 61C64630
 P 2850 5600
-F 0 "J11" H 3100 6000 50  0000 C CNN
+F 0 "J10" H 3100 6000 50  0000 C CNN
 F 1 "Conn_01x06_Male" H 3100 5900 50  0000 C CNN
 F 2 "Connector_Molex:Molex_KK-254_AE-6410-06A_1x06_P2.54mm_Vertical" H 2850 5600 50  0001 C CNN
@@
 	3750 6400 3750 4850
 $Comp
-L Connector:Conn_01x06_Male J6
+L Connector:Conn_01x06_Male J5
 U 1 1 61C2A57A
 P 1450 1600
-F 0 "J6" H 1700 2000 50  0000 C CNN
+F 0 "J5" H 1700 2000 50  0000 C CNN
 F 1 "Conn_01x06_Male" H 1700 1900 50  0000 C CNN
 F 2 "Connector_Molex:Molex_KK-254_AE-6410-06A_1x06_P2.54mm_Vertical" H 1450 1600 50  0001 C CNN
@@
 $EndComp
 $Comp
-L Connector:Conn_01x03_Female J12
+L Connector:Conn_01x03_Female J11
 U 1 1 61C6F8C4
 P 5350 1700
-F 0 "J12" H 4950 2050 50  0000 L CNN
+F 0 "J11" H 4950 2050 50  0000 L CNN
 F 1 "Conn_01x03_Female" H 4650 1950 50  0000 L CNN
 F 2 "Connector:FanPinHeader_1x03_P2.54mm_Vertical" H 5350 1700 50  0001 C CNN
@@
 $EndComp
 $Comp
-L Sensor:DHT11 U7
+L Sensor:DHT11 U8
 U 1 1 61C728C4
 P 6400 1650
-F 0 "U7" H 6156 1696 50  0000 R CNN
+F 0 "U8" H 6156 1696 50  0000 R CNN
 F 1 "DHT11" H 6156 1605 50  0000 R CNN
 F 2 "Sensor:Aosong_DHT11_5.5x12.0_P2.54mm" H 6400 1250 50  0001 C CNN
@@
 $EndComp
 $Comp
-L power:GND #PWR0140
+L power:GND #PWR051
 U 1 1 61C7572B
 P 6400 2050
-F 0 "#PWR0140" H 6400 1800 50  0001 C CNN
+F 0 "#PWR051" H 6400 1800 50  0001 C CNN
 F 1 "GND" H 6405 1877 50  0000 C CNN
 F 2 "" H 6400 2050 50  0001 C CNN
@@
 Pin 1 - Power (brown wire)\nPin 2 - Ground (black wire) \nPin 3 - Signal (blue wire)\nPin 4 not connected
 $Comp
-L power:GND #PWR0141
+L power:GND #PWR049
 U 1 1 61C789C3
 P 4950 1700
-F 0 "#PWR0141" H 4950 1450 50  0001 C CNN
+F 0 "#PWR049" H 4950 1450 50  0001 C CNN
 F 1 "GND" V 4955 1572 50  0000 R CNN
 F 2 "" H 4950 1700 50  0001 C CNN
@@
 	4950 1700 5150 1700
 $Comp
-L power:+5V #PWR0142
+L power:+5V #PWR040
 U 1 1 61C90CFA
 P 2200 1250
-F 0 "#PWR0142" H 2200 1100 50  0001 C CNN
+F 0 "#PWR040" H 2200 1100 50  0001 C CNN
 F 1 "+5V" H 2215 1423 50  0000 C CNN
 F 2 "" H 2200 1250 50  0001 C CNN
@@
 	1650 1400 2200 1400
 $Comp
-L power:+5V #PWR0143
+L power:+5V #PWR046
 U 1 1 61C92B2A
 P 3600 1250
-F 0 "#PWR0143" H 3600 1100 50  0001 C CNN
+F 0 "#PWR046" H 3600 1100 50  0001 C CNN
 F 1 "+5V" H 3615 1423 50  0000 C CNN
 F 2 "" H 3600 1250 50  0001 C CNN
@@
 	3600 1400 3600 1250
 $Comp
-L power:+5V #PWR0144
+L power:+5V #PWR041
 U 1 1 61C95B54
 P 2200 3350
-F 0 "#PWR0144" H 2200 3200 50  0001 C CNN
+F 0 "#PWR041" H 2200 3200 50  0001 C CNN
 F 1 "+5V" H 2215 3523 50  0000 C CNN
 F 2 "" H 2200 3350 50  0001 C CNN
@@
 $EndComp
 $Comp
-L power:+5V #PWR0145
+L power:+5V #PWR047
 U 1 1 61C960FB
 P 3600 3350
-F 0 "#PWR0145" H 3600 3200 50  0001 C CNN
+F 0 "#PWR047" H 3600 3200 50  0001 C CNN
 F 1 "+5V" H 3615 3523 50  0000 C CNN
 F 2 "" H 3600 3350 50  0001 C CNN
@@
 $EndComp
 $Comp
-L power:+5V #PWR0146
+L power:+5V #PWR042
 U 1 1 61C966FF
 P 2200 5350
-F 0 "#PWR0146" H 2200 5200 50  0001 C CNN
+F 0 "#PWR042" H 2200 5200 50  0001 C CNN
 F 1 "+5V" H 2215 5523 50  0000 C CNN
 F 2 "" H 2200 5350 50  0001 C CNN
@@
 $EndComp
 $Comp
-L power:+5V #PWR0147
+L power:+5V #PWR048
 U 1 1 61C96BA5
 P 3600 5350
-F 0 "#PWR0147" H 3600 5200 50  0001 C CNN
+F 0 "#PWR048" H 3600 5200 50  0001 C CNN
 F 1 "+5V" H 3615 5523 50  0000 C CNN
 F 2 "" H 3600 5350 50  0001 C CNN
@@
 	5150 1600 5050 1600
 $Comp
-L power:+5V #PWR0148
+L power:+5V #PWR050
 U 1 1 61C9C239
 P 6400 1250
-F 0 "#PWR0148" H 6400 1100 50  0001 C CNN
+F 0 "#PWR050" H 6400 1100 50  0001 C CNN
 F 1 "+5V" H 6415 1423 50  0000 C CNN
 F 2 "" H 6400 1250 50  0001 C CNN
@@
 CO_ANALOG_AUX
 $Comp
-L power:GND #PWR0149
+L power:GND #PWR037
 U 1 1 61CE7471
 P 1700 1950
-F 0 "#PWR0149" H 1700 1700 50  0001 C CNN
+F 0 "#PWR037" H 1700 1700 50  0001 C CNN
 F 1 "GND" H 1705 1777 50  0000 C CNN
 F 2 "" H 1700 1950 50  0001 C CNN
@@
 Connection ~ 3100 1700
 $Comp
-L power:GND #PWR0150
+L power:GND #PWR045
 U 1 1 61CF5F42
 P 3150 2000
-F 0 "#PWR0150" H 3150 1750 50  0001 C CNN
+F 0 "#PWR045" H 3150 1750 50  0001 C CNN
 F 1 "GND" H 3155 1827 50  0000 C CNN
 F 2 "" H 3150 2000 50  0001 C CNN
@@
 Connection ~ 1700 3750
 $Comp
-L power:GND #PWR0151
+L power:GND #PWR038
 U 1 1 61CFC141
 P 1700 4000
-F 0 "#PWR0151" H 1700 3750 50  0001 C CNN
+F 0 "#PWR038" H 1700 3750 50  0001 C CNN
 F 1 "GND" H 1705 3827 50  0000 C CNN
 F 2 "" H 1700 4000 50  0001 C CNN
@@
 Connection ~ 3100 3950
 $Comp
-L power:GND #PWR0152
+L power:GND #PWR043
 U 1 1 61D036A9
 P 3100 4000
-F 0 "#PWR0152" H 3100 3750 50  0001 C CNN
+F 0 "#PWR043" H 3100 3750 50  0001 C CNN
 F 1 "GND" H 3105 3827 50  0000 C CNN
 F 2 "" H 3100 4000 50  0001 C CNN
@@
 Connection ~ 1700 5700
 $Comp
-L power:GND #PWR0153
+L power:GND #PWR039
 U 1 1 61D0815C
 P 1700 5950
-F 0 "#PWR0153" H 1700 5700 50  0001 C CNN
+F 0 "#PWR039" H 1700 5700 50  0001 C CNN
 F 1 "GND" H 1705 5777 50  0000 C CNN
 F 2 "" H 1700 5950 50  0001 C CNN
@@
 Connection ~ 3100 5900
 $Comp
-L power:GND #PWR0154
+L power:GND #PWR044
 U 1 1 61D10D52
 P 3100 5950
-F 0 "#PWR0154" H 3100 5700 50  0001 C CNN
+F 0 "#PWR044" H 3100 5700 50  0001 C CNN
 F 1 "GND" H 3105 5777 50  0000 C CNN
 F 2 "" H 3100 5950 50  0001 C CNN
